File: stknx.kicad_pcb (KiCad board)
At the start: 0 parts

Commit message: Rough component placement
Parts:
- added C1: 1nF DNP, Capacitor_SMD:C_0402_1005Metric, F.Cu at (189.7, 113.6)
- added C10: 10uF 25V, Capacitor_SMD:C_1206_3216Metric, F.Cu at (173.9, 106.0)
- added C11: 220n 6.3V, Capacitor_SMD:C_0402_1005Metric, F.Cu at (172.5, 115.9)
- added C12: 150pF 16V, Capacitor_SMD:C_0402_1005Metric, F.Cu at (167.6, 116.4)
- added C13: 10u 35V, Capacitor_SMD:C_1206_3216Metric, F.Cu at (172.2, 111.6)
- added C14: 100n, Capacitor_SMD:C_0402_1005Metric, F.Cu at (177.2, 114.7)
- added C15: 100n, Capacitor_SMD:C_0402_1005Metric, F.Cu at (175.2, 114.4)
- added C16: 4.7u, Capacitor_SMD:C_0805_2012Metric, F.Cu at (174.8, 115.9)
- added C17: 22u 25V, Capacitor_SMD:C_1210_3225Metric, F.Cu at (168.6, 114.1)
- added C18: 1nF, Capacitor_SMD:C_0402_1005Metric, B.Cu at (161.3, 105.7)
- added C2: 220u 35V, Capacitor_SMD:C_Elec_10x10.2, F.Cu at (187.7, 102.2)
- added C3: 220u 35V, Capacitor_SMD:C_Elec_10x10.2, F.Cu at (167.3, 102.2)
- added C4: 470nF 35V, Capacitor_SMD:C_0805_2012Metric, F.Cu at (180.2, 106.5)
- added C5: 10nF 50V, Capacitor_SMD:C_0402_1005Metric, F.Cu at (179.8, 112.0)
- added C6: 100n 50V, Capacitor_SMD:C_0603_1608Metric, F.Cu at (182.3, 110.8)
- added C7: 47nF 35V, Capacitor_SMD:C_0402_1005Metric, F.Cu at (178.1, 107.5)
- added C8: 100n 50V, Capacitor_SMD:C_0603_1608Metric, F.Cu at (182.3, 108.8)
- added C9: 47nF 35V, Capacitor_SMD:C_0402_1005Metric, F.Cu at (179.4, 108.0)
- added D1: SMAJ40CA, Diode_SMD:D_SMA, F.Cu at (192.6, 111.2)
- added D2: LL4148-GS18, Diode_SMD:D_MiniMELF, F.Cu at (181.6, 115.8)
- added D3: LL4148-GS18, Diode_SMD:D_MiniMELF, F.Cu at (176.4, 105.3)
- added D4: LL4148-GS18, Diode_SMD:D_MiniMELF, F.Cu at (181.6, 113.6)
- added D5: BAT54 DNP, Diode_SMD:D_SOD-323F, B.Cu at (161.8, 107.9)
- added J1: KNX, stknx:WAGO_243-211, F.Cu at (198.7, 110.2)
- added J2: PMOD, Connector_PinHeader_2.54mm:PinHeader_1x06_P2.54mm_Horizontal, F.Cu at (158.5, 113.3)
- added J3: VDDHV, Connector_PinHeader_2.54mm:PinHeader_1x02_P2.54mm_Vertical, F.Cu at (176.2, 98.6)
- added J4: VCCCORE, Connector_PinHeader_2.54mm:PinHeader_1x02_P2.54mm_Vertical, F.Cu at (164.4, 111.6)
- added J5: VDCDC, Connector_PinHeader_2.54mm:PinHeader_1x02_P2.54mm_Vertical, F.Cu at (164.4, 115.2)
- added JP1: DCDC, Jumper:SolderJumper-3_P1.3mm_Bridged12_RoundedPad1.0x1.5mm_NumberLabels, B.Cu at (173.4, 107.0)
- added JP2: HV, Jumper:SolderJumper-2_P1.3mm_Bridged_RoundedPad1.0x1.5mm, B.Cu at (171.6, 109.8)
- added JP3: DCDC, Jumper:SolderJumper-2_P1.3mm_Open_RoundedPad1.0x1.5mm, B.Cu at (171.6, 114.8)
- added JP4: OFF, Jumper:SolderJumper-2_P1.3mm_Open_RoundedPad1.0x1.5mm, B.Cu at (171.6, 112.3)
- added JP5: LINEAR, Jumper:SolderJumper-3_P1.3mm_Bridged12_RoundedPad1.0x1.5mm_NumberLabels, B.Cu at (180.3, 114.2)
- added JP6: VCC, Jumper:SolderJumper-2_P1.3mm_Open_RoundedPad1.0x1.5mm, B.Cu at (162.1, 100.6)
- added L1: 33uH, stknx:L_WE_LQS_4012, F.Cu at (168.6, 110.3)
- added R1: 0, Resistor_SMD:R_0402_1005Metric, F.Cu at (195.5, 114.1)
- added R10: 40.2K, Resistor_SMD:R_0402_1005Metric, F.Cu at (169.7, 116.4)
- added R11: 0, Resistor_SMD:R_0402_1005Metric, F.Cu at (178.2, 114.7)
- added R12: 470K DNP, Resistor_SMD:R_0402_1005Metric, B.Cu at (163.3, 107.3)
- added R2: 10K, Resistor_SMD:R_0402_1005Metric, B.Cu at (172.1, 104.7)
- added R3: 4.7M, Resistor_SMD:R_0402_1005Metric, F.Cu at (190.2, 111.2)
- added R4: 18K DNP, Resistor_SMD:R_0402_1005Metric, F.Cu at (189.7, 112.6)
- added R5: 68, Resistor_SMD:R_2512_6332Metric, F.Cu at (186.2, 111.5)
- added R6: 1K, Resistor_SMD:R_0402_1005Metric, F.Cu at (179.9, 110.6)
- added R7: 1K, Resistor_SMD:R_0402_1005Metric, F.Cu at (179.9, 109.1)
- added R8: 10K, Resistor_SMD:R_0402_1005Metric, B.Cu at (181.6, 112.0)
- added R9: 10K, Resistor_SMD:R_0402_1005Metric, F.Cu at (171.5, 115.9)
- added TP1: HV, TestPoint:TestPoint_Pad_D1.0mm, F.Cu at (179.0, 102.0)
- added TP2: VCCCORE, TestPoint:TestPoint_Pad_D1.0mm, F.Cu at (177.3, 116.3)
- added TP3: VCCDCDC, TestPoint:TestPoint_Pad_D1.0mm, F.Cu at (164.9, 108.7)
- added U1: STKNX, Package_DFN_QFN:VQFN-24-1EP_4x4mm_P0.5mm_EP2.45x2.45mm, F.Cu at (176.2, 111.1)
Other:
- board outline added: 51.3 x 20.3 mm
- copper layers 0 -> 2
