File: stknx.kicad_sch (KiCad schematic)
At the start: 51 parts, among them J1 KNX, J2 PMOD, J3 VDDHV, J4 VCCCORE, J5 VDCDC, U1 STKNX

Commit message: Make R5 not go up in flames once we transmit the first bit
Parts:
- R5: footprint Resistor_SMD:R_0402_1005Metric -> Resistor_SMD:R_2512_6332Metric; Manufacturer YAGEO -> Vishay Dale; Order No 13-RT0402FRE0768RLCT-ND -> 541-68.0AFCT-ND; Part Description 68 Ohms ±1% 0.063W, 1/16W Chip Resistor 0402 (1005 Metric) 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 -> 68 Ohms ±1% 1W Chip Resistor 2512 (6432 Metric) Automotive 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; Part No RT0402FRE0768RL -> CRCW251268R0FKEG
Changed lines of the file:
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@@
     (property "Reference" "R5" (id 0) (at 99.06 126.1068 90))
     (property "Value" "68" (id 1) (at 99.06 128.8819 90))
-    (property "Footprint" "Resistor_SMD:R_0402_1005Metric" (id 2) (at 99.06 130.81 0)
+    (property "Footprint" "Resistor_SMD:R_2512_6332Metric" (id 2) (at 99.06 130.81 0)
       (effects (font (size 1.27 1.27)) hide)
     )
@@
       (effects (font (size 1.27 1.27)) hide)
     )
-    (property "Manufacturer" "YAGEO" (id 4) (at 99.06 130.81 0)
-      (effects (font (size 1.27 1.27)) hide)
-    )
-    (property "Order No" "13-RT0402FRE0768RLCT-ND" (id 5) (at 99.06 130.81 0)
-      (effects (font (size 1.27 1.27)) hide)
-    )
-    (property "Part Description" "68 Ohms ±1% 0.063W, 1/16W Chip Resistor 0402 (1005 Metric)  Thin Film" (id 6) (at 99.06 130.81 0)
-      (effects (font (size 1.27 1.27)) hide)
-    )
-    (property "Part No" "RT0402FRE0768RL" (id 7) (at 99.06 130.81 0)
+    (property "Manufacturer" "Vishay Dale" (id 4) (at 99.06 130.81 0)
+      (effects (font (size 1.27 1.27)) hide)
+    )
+    (property "Order No" "541-68.0AFCT-ND" (id 5) (at 99.06 130.81 0)
+      (effects (font (size 1.27 1.27)) hide)
+    )
+    (property "Part Description" "68 Ohms ±1% 1W Chip Resistor 2512 (6432 Metric) Automotive AEC-Q200 Thick Film" (id 6) (at 99.06 130.81 0)
+      (effects (font (size 1.27 1.27)) hide)
+    )
+    (property "Part No" "CRCW251268R0FKEG" (id 7) (at 99.06 130.81 0)
       (effects (font (size 1.27 1.27)) hide)
     )
@@
     )
     (path "/5f29a5b4-6ef1-4de6-93b0-fec7fb4c53cf"
-      (reference "R5") (unit 1) (value "68") (footprint "Resistor_SMD:R_0402_1005Metric")
+      (reference "R5") (unit 1) (value "68") (footprint "Resistor_SMD:R_2512_6332Metric")
     )
     (path "/4233f80a-a0fc-4a30-8fae-a3e535878768"

Commit message: Rotate D4
Connections:
- net GND: now also D4.2 (A); no longer D4.1 (K)
- net at C5.2, U1.2 (KNX_AC): now also D4.1 (K); no longer D4.2 (A)
Other:
- moved on the sheet: D4
Changed lines of the file:
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@@
     (pin "2")
   )
-  (symbol (lib_id "Device:D_Small") (at 93.98 119.38 90) (unit 1)
+  (symbol (lib_id "Device:D_Small") (at 93.98 119.38 270) (unit 1)
     (in_bom yes) (on_board yes)
-    (property "Reference" "D4" (id 0) (at 98.5519 120.2885 90)
+    (property "Reference" "D4" (id 0) (at 95.7581 118.4715 90)
       (effects (font (size 1.27 1.27)) (justify left))
     )
-    (property "Value" "TS4148RY" (id 1) (at 106.1719 117.5134 90)
+    (property "Value" "TS4148RY" (id 1) (at 95.7581 120.6116 90)
       (effects (font (size 1.27 1.27)) (justify left))
     )

Commit message: BOM
Parts:
- C14, C15: footprint https:__media.digikey.com_pdf_Data%20Sheets_Samsung%20PDFs_CL05B104KA5NNNC_Spec.pdf -> Capacitor_SMD:C_0402_1005Metric
- D2, D3, D4: value TS4148RY -> LL4148-GS18; footprint Diode_SMD:D_MELF -> Diode_SMD:D_SOD-123F; Order No LS4448GS18GICT-ND -> LL4148-GS18CT-ND; Part Description Dioden Standard 75V 150mA Oberflächenmontage SOD-80 QuadroM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 -> Diode Standard 75V 300mA (DC) Surface Mount SOD-80 MiniMELF; Part No LS4448GS18 -> LL4148-GS18
- J2: Manufacturer (none) -> Adam Tech; Order No (none) -> 2057-PH1RB-06-UA-ND; Part Description (none) -> Connector Header Through Hole, Right Angle 6 position 0.100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; Part No (none) -> PH1RB-06-UA; Supplier (none) -> Digikey
Changed lines of the file:
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@@
     (stroke (width 0) (type default) (color 0 0 0 0))
   )
-  (polyline (pts (xy 91.44 115.57) (xy 107.95 115.57))
+  (polyline (pts (xy 91.44 115.57) (xy 109.22 115.57))
     (stroke (width 0) (type default) (color 0 0 0 0))
   )
-  (polyline (pts (xy 107.95 115.57) (xy 107.95 123.19))
+  (polyline (pts (xy 109.22 115.57) (xy 109.22 123.19))
     (stroke (width 0) (type default) (color 0 0 0 0))
   )
-  (polyline (pts (xy 107.95 123.19) (xy 91.44 123.19))
+  (polyline (pts (xy 109.22 123.19) (xy 91.44 123.19))
     (stroke (width 0) (type default) (color 0 0 0 0))
   )
@@
       (effects (font (size 1.27 1.27)) (justify left))
     )
-    (property "Value" "TS4148RY" (id 1) (at 47.4981 141.5666 90)
-      (effects (font (size 1.27 1.27)) (justify left))
-    )
-    (property "Footprint" "Diode_SMD:D_MELF" (id 2) (at 59.69 139.7 90)
+    (property "Value" "LL4148-GS18" (id 1) (at 44.3231 141.5666 90)
+      (effects (font (size 1.27 1.27)) (justify left))
+    )
+    (property "Footprint" "Diode_SMD:D_SOD-123F" (id 2) (at 59.69 139.7 90)
       (effects (font (size 1.27 1.27)) hide)
     )
@@
       (effects (font (size 1.27 1.27)) hide)
     )
-    (property "Order No" "LS4448GS18GICT-ND" (id 5) (at 59.69 139.7 0)
-      (effects (font (size 1.27 1.27)) hide)
-    )
-    (property "Part Description" "Dioden Standard 75V 150mA Oberflächenmontage SOD-80 QuadroMELF" (id 6) (at 59.69 139.7 0)
-      (effects (font (size 1.27 1.27)) hide)
-    )
-    (property "Part No" "LS4448GS18" (id 7) (at 59.69 139.7 0)
+    (property "Order No" "LL4148-GS18CT-ND" (id 5) (at 59.69 139.7 0)
+      (effects (font (size 1.27 1.27)) hide)
+    )
+    (property "Part Description" "Diode Standard 75V 300mA (DC) Surface Mount SOD-80 MiniMELF" (id 6) (at 59.69 139.7 0)
+      (effects (font (size 1.27 1.27)) hide)
+    )
+    (property "Part No" "LL4148-GS18" (id 7) (at 59.69 139.7 0)
       (effects (font (size 1.27 1.27)) hide)
     )
@@
       (effects (font (size 1.27 1.27)) (justify left))
     )
-    (property "Value" "TS4148RY" (id 1) (at 95.8466 89.6619 0)
-      (effects (font (size 1.27 1.27)) (justify left))
-    )
-    (property "Footprint" "Diode_SMD:D_MELF" (id 2) (at 93.98 87.63 90)
+    (property "Value" "LL4148-GS18" (id 1) (at 95.8466 89.6619 0)
+      (effects (font (size 1.27 1.27)) (justify left))
+    )
+    (property "Footprint" "Diode_SMD:D_SOD-123F" (id 2) (at 93.98 87.63 90)
       (effects (font (size 1.27 1.27)) hide)
     )
@@
       (effects (font (size 1.27 1.27)) hide)
     )
-    (property "Order No" "LS4448GS18GICT-ND" (id 5) (at 93.98 87.63 0)
-      (effects (font (size 1.27 1.27)) hide)
-    )
-    (property "Part Description" "Dioden Standard 75V 150mA Oberflächenmontage SOD-80 QuadroMELF" (id 6) (at 93.98 87.63 0)
-      (effects (font (size 1.27 1.27)) hide)
-    )
-    (property "Part No" "LS4448GS18" (id 7) (at 93.98 87.63 0)
+    (property "Order No" "LL4148-GS18CT-ND" (id 5) (at 93.98 87.63 0)
+      (effects (font (size 1.27 1.27)) hide)
+    )
+    (property "Part Description" "Diode Standard 75V 300mA (DC) Surface Mount SOD-80 MiniMELF" (id 6) (at 93.98 87.63 0)
+      (effects (font (size 1.27 1.27)) hide)
+    )
+    (property "Part No" "LL4148-GS18" (id 7) (at 93.98 87.63 0)
       (effects (font (size 1.27 1.27)) hide)
     )
@@
       (effects (font (size 1.27 1.27)) (justify left))
     )
-    (property "Value" "TS4148RY" (id 1) (at 95.7581 120.6116 90)
-      (effects (font (size 1.27 1.27)) (justify left))
-    )
-    (property "Footprint" "Diode_SMD:D_MELF" (id 2) (at 93.98 119.38 90)
+    (property "Value" "LL4148-GS18" (id 1) (at 95.7581 120.6116 90)
+      (effects (font (size 1.27 1.27)) (justify left))
+    )
+    (property "Footprint" "Diode_SMD:D_SOD-123F" (id 2) (at 93.98 119.38 90)
       (effects (font (size 1.27 1.27)) hide)
     )
@@
       (effects (font (size 1.27 1.27)) hide)
     )
-    (property "Order No" "LS4448GS18GICT-ND" (id 5) (at 93.98 119.38 0)
-      (effects (font (size 1.27 1.27)) hide)
-    )
-    (property "Part Description" "Dioden Standard 75V 150mA Oberflächenmontage SOD-80 QuadroMELF" (id 6) (at 93.98 119.38 0)
-      (effects (font (size 1.27 1.27)) hide)
-    )
-    (property "Part No" "LS4448GS18" (id 7) (at 93.98 119.38 0)
+    (property "Order No" "LL4148-GS18CT-ND" (id 5) (at 93.98 119.38 0)
+      (effects (font (size 1.27 1.27)) hide)
+    )
+    (property "Part Description" "Diode Standard 75V 300mA (DC) Surface Mount SOD-80 MiniMELF" (id 6) (at 93.98 119.38 0)
+      (effects (font (size 1.27 1.27)) hide)
+    )
+    (property "Part No" "LL4148-GS18" (id 7) (at 93.98 119.38 0)
       (effects (font (size 1.27 1.27)) hide)
     )
@@
       (effects (font (size 1.27 1.27)) (justify left))
     )
-    (property "Footprint" "https:__media.digikey.com_pdf_Data%20Sheets_Samsung%20PDFs_CL05B104KA5NNNC_Spec.pdf" (id 2) (at 193.04 114.3 0)
+    (property "Footprint" "Capacitor_SMD:C_0402_1005Metric" (id 2) (at 193.04 114.3 0)
       (effects (font (size 1.27 1.27)) hide)
     )
@@
       (effects (font (size 1.27 1.27)) (justify left))
     )
-    (property "Footprint" "https:__media.digikey.com_pdf_Data%20Sheets_Samsung%20PDFs_CL05B104KA5NNNC_Spec.pdf" (id 2) (at 198.12 124.46 0)
+    (property "Footprint" "Capacitor_SMD:C_0402_1005Metric" (id 2) (at 198.12 124.46 0)
       (effects (font (size 1.27 1.27)) hide)
     )
@@
     )
     (property "Datasheet" "~" (id 3) (at 274.32 25.4 0)
+      (effects (font (size 1.27 1.27)) hide)
+    )
+    (property "Manufacturer" "Adam Tech" (id 4) (at 274.32 25.4 0)
+      (effects (font (size 1.27 1.27)) hide)
+    )
+    (property "Order No" "2057-PH1RB-06-UA-ND" (id 5) (at 274.32 25.4 0)
+      (effects (font (size 1.27 1.27)) hide)
+    )
+    (property "Part Description" "Connector Header Through Hole, Right Angle 6 position 0.100\" (2.54mm)" (id 6) (at 274.32 25.4 0)
+      (effects (font (size 1.27 1.27)) hide)
+    )
+    (property "Part No" "PH1RB-06-UA" (id 7) (at 274.32 25.4 0)
+      (effects (font (size 1.27 1.27)) hide)
+    )
+    (property "Supplier" "Digikey" (id 8) (at 274.32 25.4 0)
       (effects (font (size 1.27 1.27)) hide)
     )
@@
     )
     (path "/22a77341-2998-4e9d-a51f-e285c66b8925"
-      (reference "C14") (unit 1) (value "100n") (footprint "https:__media.digikey.com_pdf_Data%20Sheets_Samsung%20PDFs_CL05B104KA5NNNC_Spec.pdf")
+      (reference "C14") (unit 1) (value "100n") (footprint "Capacitor_SMD:C_0402_1005Metric")
     )
     (path "/f8260a71-8493-4036-9986-587e68e40c8d"
-      (reference "C15") (unit 1) (value "100n") (footprint "https:__media.digikey.com_pdf_Data%20Sheets_Samsung%20PDFs_CL05B104KA5NNNC_Spec.pdf")
+      (reference "C15") (unit 1) (value "100n") (footprint "Capacitor_SMD:C_0402_1005Metric")
     )
     (path "/bd971365-3636-4c88-8244-302d017f9330"
@@
     )
     (path "/6775a3fe-5193-4210-b8fe-e0cb420e79de"
-      (reference "D2") (unit 1) (value "TS4148RY") (footprint "Diode_SMD:D_MELF")
+      (reference "D2") (unit 1) (value "LL4148-GS18") (footprint "Diode_SMD:D_SOD-123F")
     )
     (path "/ea5ffd93-3c11-49cc-9806-57cd2746ac8d"
-      (reference "D3") (unit 1) (value "TS4148RY") (footprint "Diode_SMD:D_MELF")
+      (reference "D3") (unit 1) (value "LL4148-GS18") (footprint "Diode_SMD:D_SOD-123F")
     )
     (path "/16a104e3-d9cd-4d22-9aec-c81bb2e92328"
-      (reference "D4") (unit 1) (value "TS4148RY") (footprint "Diode_SMD:D_MELF")
+      (reference "D4") (unit 1) (value "LL4148-GS18") (footprint "Diode_SMD:D_SOD-123F")
     )
     (path "/6d38309b-b2e2-4739-a784-65eb9ca55906"

Commit message: BAT54
Parts:
- D5: value BAT54J DNP -> BAT54 DNP; Manufacturer (none) -> Panjit International Inc.; Order No (none) -> 3757-BAT54WS_R1_00001CT-ND; Part Description (none) -> Diode Schottky 30V 200mA Surface Mount SOD-323; Part No (none) -> BAT54WS_R1_00001; Supplier (none) -> Digikey
Changed lines of the file:
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@@
       (effects (font (size 1.27 1.27)) (justify left))
     )
-    (property "Value" "BAT54J DNP" (id 1) (at 225.5521 155.5366 90)
+    (property "Value" "BAT54 DNP" (id 1) (at 225.5521 155.5366 90)
       (effects (font (size 1.27 1.27)) (justify left))
     )
@@
       (effects (font (size 1.27 1.27)) hide)
     )
-    (property "Datasheet" "https://assets.nexperia.com/documents/data-sheet/BAT54J.pdf" (id 3) (at 223.52 153.67 0)
+    (property "Datasheet" "https://www.panjit.com.tw/en/Product/downloadPDF/BAT54WS" (id 3) (at 223.52 153.67 0)
+      (effects (font (size 1.27 1.27)) hide)
+    )
+    (property "Manufacturer" "Panjit International Inc." (id 4) (at 223.52 153.67 0)
+      (effects (font (size 1.27 1.27)) hide)
+    )
+    (property "Order No" "3757-BAT54WS_R1_00001CT-ND" (id 5) (at 223.52 153.67 0)
+      (effects (font (size 1.27 1.27)) hide)
+    )
+    (property "Part Description" "Diode Schottky 30V 200mA Surface Mount SOD-323" (id 6) (at 223.52 153.67 0)
+      (effects (font (size 1.27 1.27)) hide)
+    )
+    (property "Part No" "BAT54WS_R1_00001" (id 7) (at 223.52 153.67 0)
+      (effects (font (size 1.27 1.27)) hide)
+    )
+    (property "Supplier" "Digikey" (id 8) (at 223.52 153.67 0)
       (effects (font (size 1.27 1.27)) hide)
     )
@@
     )
     (path "/6d38309b-b2e2-4739-a784-65eb9ca55906"
-      (reference "D5") (unit 1) (value "BAT54J DNP") (footprint "Diode_SMD:D_SOD-323F")
+      (reference "D5") (unit 1) (value "BAT54 DNP") (footprint "Diode_SMD:D_SOD-323F")
     )
     (path "/5c5a297e-163c-47b5-99df-fd72414c3e38"

Commit message: Inductor footprint
Parts:
- L1: footprint (none) -> stknx:L_WE_LQS_4012
Changed lines of the file:
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@@
     (property "Reference" "L1" (id 0) (at 208.28 83.2824 90))
     (property "Value" "33uH" (id 1) (at 208.28 86.0575 90))
-    (property "Footprint" "" (id 2) (at 208.28 87.63 0)
+    (property "Footprint" "stknx:L_WE_LQS_4012" (id 2) (at 208.28 87.63 0)
       (effects (font (size 1.27 1.27)) hide)
     )
@@
     )
     (path "/6dce513d-8286-4f57-8183-d6a404537720"
-      (reference "L1") (unit 1) (value "33uH") (footprint "")
+      (reference "L1") (unit 1) (value "33uH") (footprint "stknx:L_WE_LQS_4012")
     )
     (path "/3ef4990c-8bb6-42a8-8733-7a193c85edf0"

Commit message: Rough component placement
Parts:
- D2, D3, D4: footprint Diode_SMD:D_SOD-123F -> Diode_SMD:D_MiniMELF
Changed lines of the file:
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@@
       (effects (font (size 1.27 1.27)) (justify left))
     )
-    (property "Footprint" "Diode_SMD:D_SOD-123F" (id 2) (at 59.69 139.7 90)
+    (property "Footprint" "Diode_SMD:D_MiniMELF" (id 2) (at 59.69 139.7 90)
       (effects (font (size 1.27 1.27)) hide)
     )
@@
       (effects (font (size 1.27 1.27)) (justify left))
     )
-    (property "Footprint" "Diode_SMD:D_SOD-123F" (id 2) (at 93.98 87.63 90)
+    (property "Footprint" "Diode_SMD:D_MiniMELF" (id 2) (at 93.98 87.63 90)
       (effects (font (size 1.27 1.27)) hide)
     )
@@
       (effects (font (size 1.27 1.27)) (justify left))
     )
-    (property "Footprint" "Diode_SMD:D_SOD-123F" (id 2) (at 93.98 119.38 90)
+    (property "Footprint" "Diode_SMD:D_MiniMELF" (id 2) (at 93.98 119.38 90)
       (effects (font (size 1.27 1.27)) hide)
     )
@@
     )
     (path "/6775a3fe-5193-4210-b8fe-e0cb420e79de"
-      (reference "D2") (unit 1) (value "LL4148-GS18") (footprint "Diode_SMD:D_SOD-123F")
+      (reference "D2") (unit 1) (value "LL4148-GS18") (footprint "Diode_SMD:D_MiniMELF")
     )
     (path "/ea5ffd93-3c11-49cc-9806-57cd2746ac8d"
-      (reference "D3") (unit 1) (value "LL4148-GS18") (footprint "Diode_SMD:D_SOD-123F")
+      (reference "D3") (unit 1) (value "LL4148-GS18") (footprint "Diode_SMD:D_MiniMELF")
     )
     (path "/16a104e3-d9cd-4d22-9aec-c81bb2e92328"
-      (reference "D4") (unit 1) (value "LL4148-GS18") (footprint "Diode_SMD:D_SOD-123F")
+      (reference "D4") (unit 1) (value "LL4148-GS18") (footprint "Diode_SMD:D_MiniMELF")
     )
     (path "/6d38309b-b2e2-4739-a784-65eb9ca55906"

Commit message: First attempts at routing
Parts:
- removed TP1: HV, TestPoint:TestPoint_Pad_D1.0mm, symbol Connector:TestPoint
- removed TP2: VCCCORE, TestPoint:TestPoint_Pad_D1.0mm, symbol Connector:TestPoint
- removed TP3: VCCDCDC, TestPoint:TestPoint_Pad_D1.0mm, symbol Connector:TestPoint
Changed lines of the file:
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@@
-    (stroke (width 0) (type default) (color 0 0 0 0))
-  )
-  (wire (pts (xy 247.65 102.87) (xy 247.65 113.03))
     (stroke (width 0) (type default) (color 0 0 0 0))
   )
@@
     (stroke (width 0) (type default) (color 0 0 0 0))
   )
-  (wire (pts (xy 260.35 102.87) (xy 260.35 113.03))
-    (stroke (width 0) (type default) (color 0 0 0 0))
-  )
   (wire (pts (xy 264.16 33.02) (xy 269.24 33.02))
     (stroke (width 0) (type default) (color 0 0 0 0))
@@
   )
   (wire (pts (xy 269.24 50.8) (xy 266.7 50.8))
-    (stroke (width 0) (type default) (color 0 0 0 0))
-  )
-  (wire (pts (xy 273.05 102.87) (xy 273.05 113.03))
     (stroke (width 0) (type default) (color 0 0 0 0))
   )
@@
     (effects (font (size 1.27 1.27)) (justify left bottom))
   )
-  (label "VDDHV" (at 247.65 113.03 90)
-    (effects (font (size 1.27 1.27)) (justify left bottom))
-  )
   (label "KNX_TX" (at 254 148.59 180)
     (effects (font (size 1.27 1.27)) (justify right bottom))
@@
   )
   (label "VDCDC" (at 256.54 67.31 0)
-    (effects (font (size 1.27 1.27)) (justify left bottom))
-  )
-  (label "VCCCORE" (at 260.35 113.03 90)
-    (effects (font (size 1.27 1.27)) (justify left bottom))
-  )
-  (label "VDCDC" (at 273.05 113.03 90)
     (effects (font (size 1.27 1.27)) (justify left bottom))
   )
@@
     (pin "1")
     (pin "2")
-  )
-  (symbol (lib_id "Connector:TestPoint") (at 247.65 102.87 0) (unit 1)
-    (in_bom yes) (on_board yes) (fields_autoplaced)
-    (property "Reference" "TP1" (id 0) (at 249.0471 100.12 0)
-      (effects (font (size 1.27 1.27)) (justify left))
-    )
-    (property "Value" "HV" (id 1) (at 249.0471 102.8951 0)
-      (effects (font (size 1.27 1.27)) (justify left))
-    )
-    (property "Footprint" "TestPoint:TestPoint_Pad_D1.0mm" (id 2) (at 252.73 102.87 0)
-      (effects (font (size 1.27 1.27)) hide)
-    )
-    (property "Datasheet" "~" (id 3) (at 252.73 102.87 0)
-      (effects (font (size 1.27 1.27)) hide)
-    )
-    (pin "1")
-  )
-  (symbol (lib_id "Connector:TestPoint") (at 260.35 102.87 0) (unit 1)
-    (in_bom yes) (on_board yes) (fields_autoplaced)
-    (property "Reference" "TP2" (id 0) (at 261.7471 100.12 0)
-      (effects (font (size 1.27 1.27)) (justify left))
-    )
-    (property "Value" "VCCCORE" (id 1) (at 261.7471 102.8951 0)
-      (effects (font (size 1.27 1.27)) (justify left))
-    )
-    (property "Footprint" "TestPoint:TestPoint_Pad_D1.0mm" (id 2) (at 265.43 102.87 0)
-      (effects (font (size 1.27 1.27)) hide)
-    )
-    (property "Datasheet" "~" (id 3) (at 265.43 102.87 0)
-      (effects (font (size 1.27 1.27)) hide)
-    )
-    (pin "1")
-  )
-  (symbol (lib_id "Connector:TestPoint") (at 273.05 102.87 0) (unit 1)
-    (in_bom yes) (on_board yes)
-    (property "Reference" "TP3" (id 0) (at 274.4471 100.12 0)
-      (effects (font (size 1.27 1.27)) (justify left))
-    )
-    (property "Value" "VCCDCDC" (id 1) (at 274.4471 102.8951 0)
-      (effects (font (size 1.27 1.27)) (justify left))
-    )
-    (property "Footprint" "TestPoint:TestPoint_Pad_D1.0mm" (id 2) (at 278.13 102.87 0)
-      (effects (font (size 1.27 1.27)) hide)
-    )
-    (property "Datasheet" "~" (id 3) (at 278.13 102.87 0)
-      (effects (font (size 1.27 1.27)) hide)
-    )
-    (pin "1")
   )
   (symbol (lib_id "power:GND") (at 21.59 166.37 0) (unit 1)
@@
       (reference "R12") (unit 1) (value "470K DNP") (footprint "Resistor_SMD:R_0402_1005Metric")
     )
-    (path "/f5a5796c-efd5-4cc8-9f5f-d95805094f8e"
-      (reference "TP1") (unit 1) (value "HV") (footprint "TestPoint:TestPoint_Pad_D1.0mm")
-    )
-    (path "/a66ceb91-6652-426a-a37c-8e7f388cf8be"
-      (reference "TP2") (unit 1) (value "VCCCORE") (footprint "TestPoint:TestPoint_Pad_D1.0mm")
-    )
-    (path "/003cc7f0-203b-4dd3-8df3-dfceec2a32f2"
-      (reference "TP3") (unit 1) (value "VCCDCDC") (footprint "TestPoint:TestPoint_Pad_D1.0mm")
-    )
     (path "/da787c9b-2295-43fd-985b-989329ad265b"

Commit message: Remove default-jumpers and replace them with open jumpers to avoid the need to scratch around on that beatiful PCB
Parts:
- JP1, JP5: footprint Jumper:SolderJumper-3_P1.3mm_Bridged12_RoundedPad1.0x1.5mm_NumberLabels -> Jumper:SolderJumper-3_P1.3mm_Open_RoundedPad1.0x1.5mm_NumberLabels
- JP2: footprint Jumper:SolderJumper-2_P1.3mm_Bridged_RoundedPad1.0x1.5mm -> Jumper:SolderJumper-2_P1.3mm_Open_RoundedPad1.0x1.5mm
Changed lines of the file:
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@@
       (effects (font (size 1.27 1.27)) (justify right))
     )
-    (property "Footprint" "Jumper:SolderJumper-2_P1.3mm_Bridged_RoundedPad1.0x1.5mm" (id 2) (at 64.77 34.29 0)
+    (property "Footprint" "Jumper:SolderJumper-2_P1.3mm_Open_RoundedPad1.0x1.5mm" (id 2) (at 64.77 34.29 0)
       (effects (font (size 1.27 1.27)) hide)
     )
@@
     (property "Reference" "JP1" (id 0) (at 31.75 23.0844 0))
     (property "Value" "DCDC" (id 1) (at 31.75 25.8595 0))
-    (property "Footprint" "Jumper:SolderJumper-3_P1.3mm_Bridged12_RoundedPad1.0x1.5mm_NumberLabels" (id 2) (at 31.75 27.94 0)
+    (property "Footprint" "Jumper:SolderJumper-3_P1.3mm_Open_RoundedPad1.0x1.5mm_NumberLabels" (id 2) (at 31.75 27.94 0)
       (effects (font (size 1.27 1.27)) hide)
     )
@@
     (property "Reference" "JP5" (id 0) (at 128.27 23.0844 0))
     (property "Value" "LINEAR" (id 1) (at 128.27 25.8595 0))
-    (property "Footprint" "Jumper:SolderJumper-3_P1.3mm_Bridged12_RoundedPad1.0x1.5mm_NumberLabels" (id 2) (at 128.27 27.94 0)
+    (property "Footprint" "Jumper:SolderJumper-3_P1.3mm_Open_RoundedPad1.0x1.5mm_NumberLabels" (id 2) (at 128.27 27.94 0)
       (effects (font (size 1.27 1.27)) hide)
     )
@@
     )
     (path "/2cc4e73c-1d5c-40a8-be9c-ce1f97aa5872"
-      (reference "JP1") (unit 1) (value "DCDC") (footprint "Jumper:SolderJumper-3_P1.3mm_Bridged12_RoundedPad1.0x1.5mm_NumberLabels")
+      (reference "JP1") (unit 1) (value "DCDC") (footprint "Jumper:SolderJumper-3_P1.3mm_Open_RoundedPad1.0x1.5mm_NumberLabels")
     )
     (path "/a0ab6e3a-d6d5-415a-b978-c3f481a2a4b4"
-      (reference "JP2") (unit 1) (value "HV") (footprint "Jumper:SolderJumper-2_P1.3mm_Bridged_RoundedPad1.0x1.5mm")
+      (reference "JP2") (unit 1) (value "HV") (footprint "Jumper:SolderJumper-2_P1.3mm_Open_RoundedPad1.0x1.5mm")
     )
     (path "/54baac83-2742-46a7-b7db-90dd758a152f"
@@
     )
     (path "/7c3e8968-9865-4e33-bc3f-c20d3fa94916"
-      (reference "JP5") (unit 1) (value "LINEAR") (footprint "Jumper:SolderJumper-3_P1.3mm_Bridged12_RoundedPad1.0x1.5mm_NumberLabels")
+      (reference "JP5") (unit 1) (value "LINEAR") (footprint "Jumper:SolderJumper-3_P1.3mm_Open_RoundedPad1.0x1.5mm_NumberLabels")
     )
     (path "/90f958e8-221f-44fa-8c81-f550e7e7e58f"
